File: HARDWARE/Right_Bar/Right_Bar.sch (EAGLE design)
At the start: 9 parts

Commit message: renames right and left, finished left
Parts:
- removed U$6, U$7, U$8: WS2812B-PTH, SparkFun-LED:WS2812B-PTH
- added C1: 1mF, SparkFun-Capacitors:1000UF-RADIAL-5MM-25V-20%
- added J2, J3, J4, J5: (no value), SparkFun-Connectors:CONN_01OFFSET
- added J7: (no value), SparkFun-Connectors:CONN_03
- added R1: 300, SparkFun-Resistors:300OHM-0603-1/10W-1%
- added R2: (no value), SparkFun-Resistors:RESISTORAXIAL-0.3
- J1: value (none) -> TRRS; device SparkFun-Connectors:CONN_03 -> SparkFun-Connectors:AUDIO_JACK_TRRSSMD_RA
Connections:
- removed net N$3: U$4.DO, U$6.DI
- removed net N$4: U$6.DO, U$7.DI
- removed net N$5: U$7.DO, U$8.DI
- new net N$2: R1.2, R2.2, U$3.DI
- net 5V: now also C1.+, J1.TIP, J7.3; no longer J1.3, U$6.VDD, U$7.VDD, U$8.VDD
- net DI: now also J1.RING1, R1.1, R2.1; no longer U$3.DI
- net DO: now also J7.2, U$4.DO; no longer J1.2, U$8.DO
- net GND: now also C1.-, J1.EARTH, J1.RING2, J7.1; no longer J1.1, U$6.VSS, U$7.VSS, U$8.VSS
